File: Md-rev-1.kicad_pcb (KiCad board)
At the start: 2 copper layers, 71.1 x 71.1 mm, 24 parts, among them CN1 JSTPH, J1 USB_C_Receptacle_USB2.0, J2 AudioJack4_SwitchTR1, U1 MCP73831-2-OT, U2 MAX9814

Commit message: Pushing changes to main
Parts:
- C2, C3, C4, C5, C6, D1, D2, J1, R1, R2, R3, R4, R5, R6, R7, R8, U1, U2: moved to B.Cu
- moved J2 45.2 mm to (167.6, 114.3), turned to -90 degrees
- moved D2 42.7 mm to (152.4, 121.9), turned to -90 degrees
- moved C4 38.1 mm to (143.5, 105.4), turned to 0 degrees
- moved C3 36.9 mm to (143.5, 108.0), turned to 0 degrees
- moved R9 35.0 mm to (157.5, 125.7)
- moved CN1 34.9 mm to (165.1, 100.3)
- moved C1 29.7 mm to (149.9, 137.2)
- moved S1 27.4 mm to (149.9, 91.4), turned to 0 degrees
- moved R4 23.6 mm to (148.2, 122.6), turned to 0 degrees
- moved U2 22.3 mm to (149.4, 103.6), turned to 0 degrees
- moved D1 22.2 mm to (152.4, 125.7), turned to 90 degrees
- moved R3 20.5 mm to (148.2, 125.7)
- moved U1 16.1 mm to (143.5, 112.7), turned to 180 degrees
- moved C6 15.3 mm to (154.9, 104.1), turned to 90 degrees
- moved R6 13.4 mm to (154.9, 111.8), turned to -90 degrees
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Connections:
- C2 pad 1: /VBAT -> Net-(U1-V_{BAT})
- S1 pad 1: unconnected-(S1-Pad1) -> Net-(U1-V_{BAT})
- S1 pad 2: GND -> /VBAT
- S1 pad 3: /VBAT -> unconnected-(S1-Pad3)
- U1 pad 3: /VBAT -> Net-(U1-V_{BAT})
Routing:
- net /VBAT: track 107.6 -> 22.3 mm, vias 4 -> 3
- net GND: track 213.4 -> 135.5 mm, vias 5 -> 2
- net Net-(J2-PadR1): track 74.0 -> 9.33 mm
- net Net-(U2-TH): track 43.4 -> 10.4 mm, vias 2 -> 0
- net Net-(U1-V_{BAT}): track 0.00 -> 32.7 mm, vias 0 -> 1
- net /OUTPUT: track 9.09 -> 40.1 mm
- net Net-(D2-A): track 27.8 -> 3.44 mm
- net Net-(U2-BIAS): track 22.0 -> 4.37 mm, vias 3 -> 0
- net Net-(U2-MICIN): track 19.9 -> 4.50 mm
- net Net-(U2-CG): track 19.5 -> 4.08 mm, vias 2 -> 0
- net Net-(D1-K): track 15.2 -> 3.64 mm, vias 2 -> 0
- net Net-(J1-CC2): track 17.2 -> 6.89 mm
- net Net-(U2-MICBIAS): track 17.4 -> 9.02 mm
- net Net-(U1-STAT): track 29.0 -> 21.8 mm, vias 2 -> 0
- net Net-(U1-PROG): track 14.1 -> 8.88 mm
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Other:
- board size 71.1 x 71.1 mm -> 20 x 60 mm

Commit message: updated the pill branch
Parts:
- removed CN1: JSTPH, Connector_JST:JST_PH_S2B-PH-K_1x02_P2.00mm_Horizontal
- removed J2: AudioJack4_SwitchTR1, Connector_Audio:Jack_3.5mm_PJ31060-I_Horizontal

Commit message: Updated the footprint files
Parts:
- MK1: footprint Buzzer_Beeper:MagneticBuzzer_Kingstate_KCG0601 -> Buzzer_Beeper:MagneticBuzzer_Kobitone_254-EMB73-RO
Changed lines of the file:
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@@
     )
   )
-  (footprint "Buzzer_Beeper:MagneticBuzzer_Kingstate_KCG0601" (layer "F.Cu")
+  (footprint "Buzzer_Beeper:MagneticBuzzer_Kobitone_254-EMB73-RO" (layer "F.Cu")
     (at 149.2 107.95)
-    (descr "Buzzer, Elektromagnetic Beeper, Summer,")
-    (tags "Kingstate KCG0601 ")
+    (descr "MagneticBuzzer_Kobitone_254-EMB73-RO https://www.mouser.es/datasheet/2/209/joytech_11092018_KT-400379-1501513.pdf")
+    (tags "MagneticBuzzer_Kobitone_254-EMB73-RO")
     (property "Sheetfile" "Md-rev-1.kicad_sch")
     (property "Sheetname" "")
@@
     (property "ki_keywords" "capacitance condenser microphone")
     (attr through_hole)
-    (fp_text reference "MK1" (at 1.6 -4.2) (layer "F.SilkS")
+    (fp_text reference "MK1" (at 1.95 -4.55) (layer "F.SilkS")
         (effects (font (size 1 1) (thickness 0.15)))
     )
-    (fp_text value "Microphone_Condensor" (at 1.6 4.4) (layer "F.Fab")
+    (fp_text value "Microphone_Condensor" (at 1.9 5.35) (layer "F.Fab")
         (effects (font (size 1 1) (thickness 0.15)))
     )
-    (fp_text user "+" (at 0 -1.6) (layer "F.SilkS")
+    (fp_text user "+" (at -2.7 -0.05) (layer "F.SilkS")
         (effects (font (size 1 1) (thickness 0.15)))
     )
-    (fp_text user "+" (at 0 -1.6) (layer "F.Fab")
+    (fp_text user "+" (at -2.7 -0.05) (layer "F.Fab")
         (effects (font (size 1 1) (thickness 0.15)))
     )
-    (fp_text user "${REFERENCE}" (at 1.6 -4.2) (layer "F.Fab")
+    (fp_text user "${REFERENCE}" (at 1.8 -1.85) (layer "F.Fab")
         (effects (font (size 1 1) (thickness 0.15)))
     )
-    (fp_circle (center 1.6 0) (end 5 0)
+    (fp_circle (center 1.5 0) (end 4.95 0)
       (stroke (width 0.12) (type solid)) (fill none) (layer "F.SilkS"))
-    (fp_circle (center 1.6 0) (end 5.15 0)
+    (fp_circle (center 1.5 0) (end 5.1 0)
       (stroke (width 0.05) (type solid)) (fill none) (layer "F.CrtYd"))
-    (fp_circle (center 1.6 0) (end 2.4 0)
+    (fp_circle (center 1.5 0) (end 2 0)
       (stroke (width 0.1) (type solid)) (fill none) (layer "F.Fab"))
-    (fp_circle (center 1.6 0) (end 4.9 0)
+    (fp_circle (center 1.5 0) (end 4.85 0)
       (stroke (width 0.1) (type solid)) (fill none) (layer "F.Fab"))
-    (pad "1" thru_hole rect (at 0 0) (size 1.6 1.6) (drill 1) (layers "*.Cu" "*.Mask")
+    (pad "1" thru_hole rect (at 0 0) (size 2 2) (drill 0.9) (layers "*.Cu" "*.Mask")
       (net 1 "GND") (pinfunction "-") (pintype "passive"))
-    (pad "2" thru_hole circle (at 3.2 0) (size 1.6 1.6) (drill 1) (layers "*.Cu" "*.Mask")
+    (pad "2" thru_hole circle (at 3 0) (size 2 2) (drill 0.9) (layers "*.Cu" "*.Mask")
       (net 4 "Net-(MK1-+)") (pinfunction "+") (pintype "passive"))
-    (model "${KICAD6_3DMODEL_DIR}/3rd-party-imports/MIC_ELECTRET-P2,54MM-D9,7MM-H6.5MM.stp"
+    (model "${KICAD7_3DMODEL_DIR}/Buzzer_Beeper.3dshapes/MagneticBuzzer_Kobitone_254-EMB73-RO.wrl" hide
       (offset (xyz 0 0 0))
       (scale (xyz 1 1 1))
-      (rotate (xyz 0 0 90))
+      (rotate (xyz 0 0 0))
+    )
+    (model ":KICAD7_3DMODEL_DIR:3rd-party-imports/MIC_ELECTRET-P2,54MM-D9,7MM-H6.5MM.stp"
+      (offset (xyz 2.5 0 0))
+      (scale (xyz 1 1 1))
+      (rotate (xyz 0 0 -90))
     )
   )

Commit message: pushing past changes
Routing:
- net (no net): track 0.00 -> 184.9 mm, vias 0 -> 3
- net GND: track 135.5 -> 0.00 mm, vias 2 -> 0
- net /OUTPUT: track 40.1 -> 0.00 mm, vias 1 -> 0
- net Net-(J2-PadR1): track 9.33 -> 0.00 mm

Commit message: updated board
Parts:
- added CN1: JSTPH, Connector_JST:JST_PH_S2B-PH-K_1x02_P2.00mm_Horizontal, F.Cu at (168.2, 78.7)
- added J2: AudioJack4_SwitchTR1, Connector_Audio:Jack_3.5mm_PJ31060-I_Horizontal, F.Cu at (144.3, 116.1)
- C1: moved to B.Cu
- moved C1 35.0 mm to (115.2, 132.1), turned to 0 degrees
- moved D1 33.0 mm to (119.4, 125.7)
- moved D2 33.0 mm to (119.4, 121.9)
- moved C2 33.0 mm to (114.3, 119.4)
- moved C3 33.0 mm to (110.5, 108.0)
- moved C4 33.0 mm to (110.5, 105.4)
- moved C5 33.0 mm to (121.9, 100.3)
- moved C6 33.0 mm to (121.9, 104.1)
- moved R1 33.0 mm to (110.1, 125.7)
- moved R2 33.0 mm to (110.1, 122.6)
- moved R5 33.0 mm to (110.1, 119.4)
- moved R6 33.0 mm to (121.9, 111.8)
- moved R7 33.0 mm to (121.9, 108.0)
- moved R8 33.0 mm to (124.4, 108.0)
- moved R9 33.0 mm to (124.4, 125.7)
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Routing:
- net (no net): track 184.9 -> 0.00 mm, vias 3 -> 0
- net /5V: track 45.9 -> 0.00 mm
- net Net-(U1-V_{BAT}): track 32.7 -> 0.00 mm, vias 1 -> 0
- net /VBAT: track 22.3 -> 0.00 mm, vias 3 -> 0
- net Net-(U1-STAT): track 21.8 -> 3.28 mm
- net Net-(MK1-+): track 17.2 -> 0.36 mm, vias 1 -> 0
- net Net-(J1-CC1): track 12.4 -> 0.00 mm
- net Net-(U2-TH): track 10.4 -> 0.05 mm
- net GND: track 0.00 -> 10.0 mm
- net Net-(U1-PROG): track 8.88 -> 0.00 mm
- net Net-(U2-MICBIAS): track 9.02 -> 1.27 mm
- net Net-(J1-CC2): track 6.89 -> 0.00 mm
- net Net-(U2-CT): track 5.57 -> 0.00 mm
- net Net-(U2-MICIN): track 4.50 -> 0.00 mm
- net Net-(U2-BIAS): track 4.37 -> 0.00 mm
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Other:
- board size 20 x 60 mm -> 14.3 x 60.5 mm

Commit message: New meditation device layout
Parts:
- added C7: 10uF, Capacitor_SMD:C_0805_2012Metric, B.Cu at (167.5, 124.0)
- C1, C5, C6, D1, D2, J1, R3, R4, R6, R7, R8, U2: moved to F.Cu
- S1: value 500SSP1S1M6QEA -> 500ASSP1SM6QE; footprint 500SSP1S1M6QEA:SW_500SSP1S1M6QEA -> 500ASSP1SM6QE:SW_500ASSP1SM6QE
- moved CN1 136.3 mm to (67.3, 170.4)
- moved R9 95.7 mm to (219.6, 136.0), turned to 180 degrees
- moved C5 59.6 mm to (176.5, 124.4), turned to 180 degrees
- moved C6 54.6 mm to (172.6, 124.4), turned to 0 degrees
- moved R8 53.6 mm to (176.4, 121.1), turned to 180 degrees
- moved U2 53.0 mm to (166.7, 120.2)
- moved R7 52.3 mm to (172.6, 121.1), turned to 180 degrees
- moved R6 51.0 mm to (172.5, 117.9), turned to 180 degrees
- moved U1 43.0 mm to (148.7, 132.4), turned to 0 degrees
- moved C3 41.5 mm to (141.0, 136.1), turned to 90 degrees
- moved C4 41.0 mm to (137.6, 136.2), turned to 90 degrees
- moved R5 38.1 mm to (144.3, 136.1), turned to 90 degrees
- moved R2 35.6 mm to (144.3, 132.4), turned to -90 degrees
- moved R1 31.6 mm to (141.0, 132.4), turned to -90 degrees
- moved R4 31.0 mm to (146.2, 122.7), turned to 90 degrees
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Connections:
- CN1 pad 2: /VBAT -> /GAIN
- S1 pad 2: /VBAT -> /GAIN
- U2 pad 2: /VBAT -> /GAIN
- U2 pad 5: /VBAT -> /GAIN
- U2 pad 6: /OUTPUT -> Net-(U2-MICOUT)
Routing:
- net GND: track 10.0 -> 62.0 mm, vias 0 -> 1
- net /5V: track 0.00 -> 23.3 mm
- net Net-(J2-PadR1): track 0.00 -> 15.6 mm, vias 0 -> 1
- net Net-(D1-K): track 3.64 -> 15.6 mm
- net Net-(U2-MICIN): track 0.00 -> 9.58 mm
- net Net-(D2-A): track 3.44 -> 11.6 mm
- net Net-(U2-MICBIAS): track 1.27 -> 8.68 mm
- net Net-(U2-BIAS): track 0.00 -> 6.86 mm
- net Net-(U2-TH): track 0.05 -> 6.83 mm
- net Net-(U1-STAT): track 3.28 -> 9.93 mm
- net Net-(MK1-+): track 0.36 -> 3.30 mm
- net /GAIN: track 0.00 -> 1.00 mm
Other:
- board size 14.3 x 60.5 mm -> 50 x 21.5 mm
