File: Md-rev-1.kicad_sch (KiCad schematic)
At the start: 28 parts, among them CN2 JSTPH, J1 USB_C_Receptacle_USB2.0, J2 54-00177, U1 MCP73831-2-OT, U2 max9814etd+t

Commit message: final save
Changed lines of the file:
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@@
   (junction (at 82.55 120.65) (diameter 0) (color 0 0 0 0)
   )
-  (junction (at 154.94 140.97) (diameter 0) (color 0 0 0 0)
-  )
   (junction (at 281.94 102.87) (diameter 0) (color 0 0 0 0)
   )
@@
   )
   (junction (at 347.98 119.38) (diameter 0) (color 0 0 0 0)
+  )
+  (junction (at 157.48 127) (diameter 0) (color 0 0 0 0)
   )
   (junction (at 34.29 148.59) (diameter 0) (color 0 0 0 0)
@@
     (stroke (width 0.1524) (type solid))
   )
+  (wire (pts (xy 157.48 127) (xy 166.37 127))
+    (stroke (width 0) (type default))
+  )
   (wire (pts (xy 179.07 97.79) (xy 179.07 100.33))
     (stroke (width 0) (type default))
@@
     (stroke (width 0) (type default))
   )
-  (wire (pts (xy 154.94 140.97) (xy 154.94 153.67))
-    (stroke (width 0) (type default))
-  )
   (wire (pts (xy 200.66 97.79) (xy 209.55 97.79))
     (stroke (width 0) (type default))
   )
-  (wire (pts (xy 154.94 129.54) (xy 154.94 140.97))
+  (wire (pts (xy 154.94 129.54) (xy 154.94 153.67))
     (stroke (width 0) (type default))
   )
@@
     (stroke (width 0) (type default))
   )
-  (wire (pts (xy 154.94 127) (xy 166.37 127))
+  (wire (pts (xy 154.94 127) (xy 157.48 127))
     (stroke (width 0) (type default))
   )
@@
     )
   )
-  (symbol (lib_id "power:PWR_FLAG") (at 154.94 140.97 90) (unit 1)
-    (in_bom yes) (on_board yes) (dnp no)
-    (property "Reference" "#FLG02" (at 153.035 140.97 0)
-      (effects (font (size 1.27 1.27)) hide)
-    )
-    (property "Value" "PWR_FLAG" (at 149.86 140.97 90)
-      (effects (font (size 1.27 1.27)) (justify left))
-    )
-    (property "Footprint" "" (at 154.94 140.97 0)
-      (effects (font (size 1.27 1.27)) hide)
-    )
-    (property "Datasheet" "~" (at 154.94 140.97 0)
-      (effects (font (size 1.27 1.27)) hide)
-    )
-    (pin "1")
-    (instances
-      (project "Md-rev-1"
-        (path "/34e1f0a2-75b5-46dc-b967-b4433c15cc45"
-          (reference "#FLG02") (unit 1)
-        )
-      )
-    )
-  )
   (symbol (lib_id "power:GND") (at 154.94 153.67 0) (unit 1)
     (in_bom yes) (on_board yes) (dnp no) (fields_autoplaced)
@@
   )
   (symbol (lib_id "500ASSP1SM6QE:500ASSP1SM6QE") (at 147.32 127 180) (unit 1)
-    (in_bom yes) (on_board yes) (dnp no) (fields_autoplaced)
-    (property "Reference" "S1" (at 147.32 119.38 0)
-      (effects (font (size 1.27 1.27)))
-    )
-    (property "Value" "500ASSP1SM6QE" (at 147.32 121.92 0)
+    (in_bom yes) (on_board yes) (dnp no)
+    (property "Reference" "S1" (at 147.32 116.84 0)
+      (effects (font (size 1.27 1.27)))
+    )
+    (property "Value" "500ASSP1SM6QE" (at 147.32 119.38 0)
       (effects (font (size 1.27 1.27)))
     )
@@
         )
       )
+    )
+  )
+  (symbol (lib_id "power:PWR_FLAG") (at 157.48 127 0) (unit 1)
+    (in_bom yes) (on_board yes) (dnp no)
+    (property "Reference" "#FLG02" (at 157.48 125.095 0)
+      (effects (font (size 1.27 1.27)) hide)
+    )
+    (property "Value" "PWR_FLAG" (at 149.86 123.19 0)
+      (effects (font (size 1.27 1.27)) (justify left))
+    )
+    (property "Footprint" "" (at 157.48 127 0)
+      (effects (font (size 1.27 1.27)) hide)
+    )
+    (property "Datasheet" "~" (at 157.48 127 0)
+      (effects (font (size 1.27 1.27)) hide)
+    )
+    (pin "1")
+    (instances
+      (project "Md-rev-1"
+        (path "/34e1f0a2-75b5-46dc-b967-b4433c15cc45"
+          (reference "#FLG02") (unit 1)
+        )
+      )

Commit message: updated the schematic and the PCB
Connections:
- net VDD: no longer C7.2, MK1.2, R6.1
- new net: C7.2, MK1.2, R6.1
Other:
- moved on the sheet: C7
Changed lines of the file:
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@@
   (junction (at 200.66 125.73) (diameter 0) (color 0 0 0 0)
-  )
-  (junction (at 271.78 115.57) (diameter 0) (color 0 0 0 0)
   )
   (junction (at 200.66 107.95) (diameter 0) (color 0 0 0 0)
@@
     (stroke (width 0) (type default))
   )
-  (wire (pts (xy 260.35 115.57) (xy 264.16 115.57))
+  (wire (pts (xy 260.35 115.57) (xy 262.89 115.57))
     (stroke (width 0) (type default))
   )
@@
   )
   (wire (pts (xy 82.55 110.49) (xy 82.55 120.65))
+    (stroke (width 0) (type default))
+  )
+  (wire (pts (xy 271.78 110.49) (xy 271.78 125.73))
     (stroke (width 0) (type default))
   )
@@
     (stroke (width 0) (type default))
   )
-  (wire (pts (xy 271.78 115.57) (xy 281.94 115.57))
+  (wire (pts (xy 270.51 115.57) (xy 281.94 115.57))
     (stroke (width 0) (type default))
   )
@@
     (stroke (width 0.1524) (type solid))
   )
-  (wire (pts (xy 271.78 110.49) (xy 271.78 115.57))
-    (stroke (width 0) (type default))
-  )
   (wire (pts (xy 100.33 110.49) (xy 105.41 110.49))
     (stroke (width 0) (type default))
@@
   )
   (wire (pts (xy 200.66 139.7) (xy 233.68 139.7))
-    (stroke (width 0) (type default))
-  )
-  (wire (pts (xy 271.78 115.57) (xy 271.78 125.73))
     (stroke (width 0) (type default))
   )
@@
     )
   )
-  (symbol (lib_id "Device:C") (at 267.97 115.57 90) (unit 1)
+  (symbol (lib_id "Device:C") (at 266.7 115.57 90) (unit 1)
     (in_bom yes) (on_board yes) (dnp no)
-    (property "Reference" "C7" (at 264.16 114.3 90)
-      (effects (font (size 1.27 1.27)))
-    )
-    (property "Value" "0.1uF" (at 264.16 116.84 90)
-      (effects (font (size 1.27 1.27)))
-    )
-    (property "Footprint" "Capacitor_SMD:C_0805_2012Metric" (at 271.78 114.6048 0)
-      (effects (font (size 1.27 1.27)) hide)
-    )
-    (property "Datasheet" "~" (at 267.97 115.57 0)
-      (effects (font (size 1.27 1.27)) hide)
-    )
+    (property "Reference" "C7" (at 262.89 114.3 90)
+      (effects (font (size 1.27 1.27)))
+    )
+    (property "Value" "0.1uF" (at 262.89 116.84 90)
+      (effects (font (size 1.27 1.27)))
+    )
+    (property "Footprint" "Capacitor_SMD:C_0805_2012Metric" (at 270.51 114.6048 0)
+      (effects (font (size 1.27 1.27)) hide)
+    )
+    (property "Datasheet" "~" (at 266.7 115.57 0)
+      (effects (font (size 1.27 1.27)) hide)
+    )
